Commit message: set request.format_result_as_input = false to debug the collision in 2d and 3d successfully

File: support/urdf/2d_obstacle_robot.urdf (robot description, URDF)
Before this commit: robot two_d_obstacle_robot, 4 links, 3 joints
Joints:
- joint joint_x: origin xyz=1.0 0.78 0 rpy=0 0 0 -> xyz=0 0 0 rpy=0 0 0
- joint obstacle_joint: origin xyz=1.0 0.45 0.0 rpy=0 0 0 -> xyz=1.0 0.78 0.0 rpy=0 0 0

Commit message: 3d example with subgoal and obstacle checking between start and subgoal

File: support/urdf/2d_obstacle_robot.urdf (robot description, URDF)
Before this commit: robot two_d_obstacle_robot, 4 links, 3 joints
Joints:
- joint obstacle_joint: origin xyz=1.0 0.78 0.0 rpy=0 0 0 -> xyz=1.0 0.6 0.0 rpy=0 0 0

File: support/urdf/three_d_robot.urdf (robot description, URDF)
Before this commit: robot three_d_robot, 5 links, 4 joints
Links:
- removed link link_x
- removed link link_y
- added link x_link
- added link y_link
Joints:
- joint joint_x: child link_x -> x_link; limit lower=-5.0 upper=5.0 effort=10.0 velocity=2.0 -> lower=-10.0 upper=10.0 effort=100 velocity=10
- joint joint_y: child link_y -> y_link; limit lower=-5.0 upper=5.0 effort=10.0 velocity=2.0 -> lower=-10.0 upper=10.0 effort=100 velocity=10; parent link_x -> x_link
- joint joint_z: limit lower=-2.0 upper=2.0 effort=10.0 velocity=2.0 -> lower=-2.0 upper=2.0 effort=100 velocity=10; parent link_y -> y_link
- joint obstacle_joint: origin xyz=1.0 0.6 0.0 rpy=0 0 0 -> xyz=0.5 0.6 0.0 rpy=0 0 0
